Commit message: adjusted joint limits and mass

File: humanoid_final_copy_description/urdf/humanoid_final_copy_backup.xacro (robot description, xacro)
@@ -1,7 +1,7 @@
 <?xml version="1.0" ?>
 <robot name="humanoid_final_copy" xmlns:xacro="http://www.ros.org/wiki/xacro">
-<xacro:include filename="/home/ubuntu/ethr_rc_robot_assets/humanoid-description/humanoid_final_copy_description/urdf/materials.xacro" />
-<xacro:include filename="/home/ubuntu/ethr_rc_robot_assets/humanoid-description/humanoid_final_copy_description/urdf/humanoid_final_copy.trans" />
-<xacro:include filename="/home/ubuntu/ethr_rc_robot_assets/humanoid-description/humanoid_final_copy_description/urdf/humanoid_final_copy.gazebo" />
+<xacro:include filename="$(find humanoid_final_copy_description)/urdf/materials.xacro" />
+<xacro:include filename="$(find humanoid_final_copy_description)/urdf/humanoid_final_copy.trans" />
+<xacro:include filename="$(find humanoid_final_copy_description)/urdf/humanoid_final_copy.gazebo" />
 <link name="base_link">
   <inertial>
@@ -13,5 +13,5 @@
     <origin xyz="0 0 0" rpy="0 0 0"/>
     <geometry>
-      <mesh filename="file:///home/ubuntu/ethr_rc_robot_assets/humanoid-description/humanoid_final_copy_description/meshes/base_link.stl" scale="0.001 0.001 0.001"/>
+      <mesh filename="file://$(find humanoid_final_copy_description)/meshes/base_link.stl" scale="0.001 0.001 0.001"/>
     </geometry>
     <material name="silver"/>
@@ -20,5 +20,5 @@
     <origin xyz="0 0 0" rpy="0 0 0"/>
     <geometry>
-      <mesh filename="file:///home/ubuntu/ethr_rc_robot_assets/humanoid-description/humanoid_final_copy_description/meshes/base_link.stl" scale="0.001 0.001 0.001"/>
+      <mesh filename="file://$(find humanoid_final_copy_description)/meshes/base_link.stl" scale="0.001 0.001 0.001"/>
     </geometry>
   </collision>
@@ -33,5 +33,5 @@
     <origin xyz="-0.199791 -0.054809 -0.230171" rpy="0 0 0"/>
     <geometry>
-      <mesh filename="file:///home/ubuntu/ethr_rc_robot_assets/humanoid-description/humanoid_final_copy_description/meshes/shoulder_upper_left_1.stl" scale="0.001 0.001 0.001"/>
+      <mesh filename="file://$(find humanoid_final_copy_description)/meshes/shoulder_upper_left_1.stl" scale="0.001 0.001 0.001"/>
     </geometry>
     <material name="silver"/>
@@ -40,5 +40,5 @@
     <origin xyz="-0.199791 -0.054809 -0.230171" rpy="0 0 0"/>
     <geometry>
-      <mesh filename="file:///home/ubuntu/ethr_rc_robot_assets/humanoid-description/humanoid_final_copy_description/meshes/shoulder_upper_left_1.stl" scale="0.001 0.001 0.001"/>
+      <mesh filename="file://$(find humanoid_final_copy_description)/meshes/shoulder_upper_left_1.stl" scale="0.001 0.001 0.001"/>
     </geometry>
   </collision>
@@ -53,5 +53,5 @@
     <origin xyz="0.06006 -0.100063 -0.434577" rpy="0 0 0"/>
     <geometry>
-      <mesh filename="file:///home/ubuntu/ethr_rc_robot_assets/humanoid-description/humanoid_final_copy_description/meshes/motor_2_left_1.stl" scale="0.001 0.001 0.001"/>
+      <mesh filename="file://$(find humanoid_final_copy_description)/meshes/motor_2_left_1.stl" scale="0.001 0.001 0.001"/>
     </geometry>
     <material name="silver"/>
@@ -60,5 +60,5 @@
     <origin xyz="0.06006 -0.100063 -0.434577" rpy="0 0 0"/>
     <geometry>
-      <mesh filename="file:///home/ubuntu/ethr_rc_robot_assets/humanoid-description/humanoid_final_copy_description/meshes/motor_2_left_1.stl" scale="0.001 0.001 0.001"/>
+      <mesh filename="file://$(find humanoid_final_copy_description)/meshes/motor_2_left_1.stl" scale="0.001 0.001 0.001"/>
     </geometry>
   </collision>
@@ -73,5 +73,5 @@
     <origin xyz="-0.243413 -0.015939 -0.262343" rpy="0 0 0"/>
     <geometry>
-      <mesh filename="file:///home/ubuntu/ethr_rc_robot_assets/humanoid-description/humanoid_final_copy_description/meshes/shoulder_lower_left_1.stl" scale="0.001 0.001 0.001"/>
+      <mesh filename="file://$(find humanoid_final_copy_description)/meshes/shoulder_lower_left_1.stl" scale="0.001 0.001 0.001"/>
     </geometry>
     <material name="silver"/>
@@ -80,5 +80,5 @@
     <origin xyz="-0.243413 -0.015939 -0.262343" rpy="0 0 0"/>
     <geometry>
-      <mesh filename="file:///home/ubuntu/ethr_rc_robot_assets/humanoid-description/humanoid_final_copy_description/meshes/shoulder_lower_left_1.stl" scale="0.001 0.001 0.001"/>
+      <mesh filename="file://$(find humanoid_final_copy_description)/meshes/shoulder_lower_left_1.stl" scale="0.001 0.001 0.001"/>
     </geometry>
   </collision>
@@ -93,5 +93,5 @@
     <origin xyz="-0.256232 -0.023115 -0.202865" rpy="0 0 0"/>
     <geometry>
-      <mesh filename="file:///home/ubuntu/ethr_rc_robot_assets/humanoid-description/humanoid_final_copy_description/meshes/motor_3_left_1.stl" scale="0.001 0.001 0.001"/>
+      <mesh filename="file://$(find humanoid_final_copy_description)/meshes/motor_3_left_1.stl" scale="0.001 0.001 0.001"/>
     </geometry>
     <material name="silver"/>
@@ -100,5 +100,5 @@
     <origin xyz="-0.256232 -0.023115 -0.202865" rpy="0 0 0"/>
     <geometry>
-      <mesh filename="file:///home/ubuntu/ethr_rc_robot_assets/humanoid-description/humanoid_final_copy_description/meshes/motor_3_left_1.stl" scale="0.001 0.001 0.001"/>
+      <mesh filename="file://$(find humanoid_final_copy_description)/meshes/motor_3_left_1.stl" scale="0.001 0.001 0.001"/>
     </geometry>
   </collision>
@@ -113,5 +113,5 @@
     <origin xyz="-0.254187 -0.017133 -0.135735" rpy="0 0 0"/>
     <geometry>
-      <mesh filename="file:///home/ubuntu/ethr_rc_robot_assets/humanoid-description/humanoid_final_copy_description/meshes/elbow_upper_left_1.stl" scale="0.001 0.001 0.001"/>
+      <mesh filename="file://$(find humanoid_final_copy_description)/meshes/elbow_upper_left_1.stl" scale="0.001 0.001 0.001"/>
     </geometry>
     <material name="silver"/>
@@ -120,5 +120,5 @@
     <origin xyz="-0.254187 -0.017133 -0.135735" rpy="0 0 0"/>
     <geometry>
-      <mesh filename="file:///home/ubuntu/ethr_rc_robot_assets/humanoid-description/humanoid_final_copy_description/meshes/elbow_upper_left_1.stl" scale="0.001 0.001 0.001"/>
+      <mesh filename="file://$(find humanoid_final_copy_description)/meshes/elbow_upper_left_1.stl" scale="0.001 0.001 0.001"/>
     </geometry>
   </collision>
@@ -133,5 +133,5 @@
     <origin xyz="-0.259849 0.033689 -0.048187" rpy="0 0 0"/>
     <geometry>
-      <mesh filename="file:///home/ubuntu/ethr_rc_robot_assets/humanoid-description/humanoid_final_copy_description/meshes/motor_4_left_1.stl" scale="0.001 0.001 0.001"/>
+      <mesh filename="file://$(find humanoid_final_copy_description)/meshes/motor_4_left_1.stl" scale="0.001 0.001 0.001"/>
     </geometry>
     <material name="silver"/>
@@ -140,5 +140,5 @@
     <origin xyz="-0.259849 0.033689 -0.048187" rpy="0 0 0"/>
     <geometry>
-      <mesh filename="file:///home/ubuntu/ethr_rc_robot_assets/humanoid-description/humanoid_final_copy_description/meshes/motor_4_left_1.stl" scale="0.001 0.001 0.001"/>
+      <mesh filename="file://$(find humanoid_final_copy_description)/meshes/motor_4_left_1.stl" scale="0.001 0.001 0.001"/>
     </geometry>
   </collision>
@@ -153,5 +153,5 @@
     <origin xyz="-0.317505 0.066303 -0.060777" rpy="0 0 0"/>
     <geometry>
-      <mesh filename="file:///home/ubuntu/ethr_rc_robot_assets/humanoid-description/humanoid_final_copy_description/meshes/elbow_lower_left_1.stl" scale="0.001 0.001 0.001"/>
+      <mesh filename="file://$(find humanoid_final_copy_description)/meshes/elbow_lower_left_1.stl" scale="0.001 0.001 0.001"/>
     </geometry>
     <material name="silver"/>
@@ -160,5 +160,5 @@
     <origin xyz="-0.317505 0.066303 -0.060777" rpy="0 0 0"/>
     <geometry>
-      <mesh filename="file:///home/ubuntu/ethr_rc_robot_assets/humanoid-description/humanoid_final_copy_description/meshes/elbow_lower_left_1.stl" scale="0.001 0.001 0.001"/>
+      <mesh filename="file://$(find humanoid_final_copy_description)/meshes/elbow_lower_left_1.stl" scale="0.001 0.001 0.001"/>
     </geometry>
   </collision>
@@ -173,5 +173,5 @@
     <origin xyz="-0.289633 0.118222 -0.028792" rpy="0 0 0"/>
     <geometry>
-      <mesh filename="file:///home/ubuntu/ethr_rc_robot_assets/humanoid-description/humanoid_final_copy_description/meshes/motor_5_left_1.stl" scale="0.001 0.001 0.001"/>
+      <mesh filename="file://$(find humanoid_final_copy_description)/meshes/motor_5_left_1.stl" scale="0.001 0.001 0.001"/>
     </geometry>
     <material name="silver"/>
@@ -180,5 +180,5 @@
     <origin xyz="-0.289633 0.118222 -0.028792" rpy="0 0 0"/>
     <geometry>
-      <mesh filename="file:///home/ubuntu/ethr_rc_robot_assets/humanoid-description/humanoid_final_copy_description/meshes/motor_5_left_1.stl" scale="0.001 0.001 0.001"/>
+      <mesh filename="file://$(find humanoid_final_copy_description)/meshes/motor_5_left_1.stl" scale="0.001 0.001 0.001"/>
     </geometry>
   </collision>
@@ -193,5 +193,5 @@
     <origin xyz="-0.303724 0.120673 0.0371" rpy="0 0 0"/>
     <geometry>
-      <mesh filename="file:///home/ubuntu/ethr_rc_robot_assets/humanoid-description/humanoid_final_copy_description/meshes/wrist_upper_left_1.stl" scale="0.001 0.001 0.001"/>
+      <mesh filename="file://$(find humanoid_final_copy_description)/meshes/wrist_upper_left_1.stl" scale="0.001 0.001 0.001"/>
     </geometry>
     <material name="silver"/>
@@ -200,5 +200,5 @@
     <origin xyz="-0.303724 0.120673 0.0371" rpy="0 0 0"/>
     <geometry>
-      <mesh filename="file:///home/ubuntu/ethr_rc_robot_assets/humanoid-description/humanoid_final_copy_description/meshes/wrist_upper_left_1.stl" scale="0.001 0.001 0.001"/>
+      <mesh filename="file://$(find humanoid_final_copy_description)/meshes/wrist_upper_left_1.stl" scale="0.001 0.001 0.001"/>
     </geometry>
   </collision>
@@ -213,5 +213,5 @@
     <origin xyz="-0.284257 0.113162 0.078158" rpy="0 0 0"/>
     <geometry>
-      <mesh filename="file:///home/ubuntu/ethr_rc_robot_assets/humanoid-description/humanoid_final_copy_description/meshes/motor_6_left_1.stl" scale="0.001 0.001 0.001"/>
+      <mesh filename="file://$(find humanoid_final_copy_description)/meshes/motor_6_left_1.stl" scale="0.001 0.001 0.001"/>
     </geometry>
     <material name="silver"/>
@@ -220,5 +220,5 @@
     <origin xyz="-0.284257 0.113162 0.078158" rpy="0 0 0"/>
     <geometry>
-      <mesh filename="file:///home/ubuntu/ethr_rc_robot_assets/humanoid-description/humanoid_final_copy_description/meshes/motor_6_left_1.stl" scale="0.001 0.001 0.001"/>
+      <mesh filename="file://$(find humanoid_final_copy_description)/meshes/motor_6_left_1.stl" scale="0.001 0.001 0.001"/>
     </geometry>
   </collision>
@@ -233,5 +233,5 @@
     <origin xyz="-0.307348 0.172729 0.056593" rpy="0 0 0"/>
     <geometry>
-      <mesh filename="file:///home/ubuntu/ethr_rc_robot_assets/humanoid-description/humanoid_final_copy_description/meshes/wrist_lower_left_1.stl" scale="0.001 0.001 0.001"/>
+      <mesh filename="file://$(find humanoid_final_copy_description)/meshes/wrist_lower_left_1.stl" scale="0.001 0.001 0.001"/>
     </geometry>
     <material name="silver"/>
@@ -240,5 +240,5 @@
     <origin xyz="-0.307348 0.172729 0.056593" rpy="0 0 0"/>
     <geometry>
-      <mesh filename="file:///home/ubuntu/ethr_rc_robot_assets/humanoid-description/humanoid_final_copy_description/meshes/wrist_lower_left_1.stl" scale="0.001 0.001 0.001"/>
+      <mesh filename="file://$(find humanoid_final_copy_description)/meshes/wrist_lower_left_1.stl" scale="0.001 0.001 0.001"/>
     </geometry>
   </collision>
@@ -253,5 +253,5 @@
     <origin xyz="-0.338511 0.16397 0.104879" rpy="0 0 0"/>
     <geometry>
-      <mesh filename="file:///home/ubuntu/ethr_rc_robot_assets/humanoid-description/humanoid_final_copy_description/meshes/motor_7_left_1.stl" scale="0.001 0.001 0.001"/>
+      <mesh filename="file://$(find humanoid_final_copy_description)/meshes/motor_7_left_1.stl" scale="0.001 0.001 0.001"/>
     </geometry>
     <material name="silver"/>
@@ -260,5 +260,5 @@
     <origin xyz="-0.338511 0.16397 0.104879" rpy="0 0 0"/>
     <geometry>
-      <mesh filename="file:///home/ubuntu/ethr_rc_robot_assets/humanoid-description/humanoid_final_copy_description/meshes/motor_7_left_1.stl" scale="0.001 0.001 0.001"/>
+      <mesh filename="file://$(find humanoid_final_copy_description)/meshes/motor_7_left_1.stl" scale="0.001 0.001 0.001"/>
     </geometry>
   </collision>
@@ -273,5 +273,5 @@
     <origin xyz="-0.356985 0.180306 0.129143" rpy="0 0 0"/>
     <geometry>
-      <mesh filename="file:///home/ubuntu/ethr_rc_robot_assets/humanoid-description/humanoid_final_copy_description/meshes/eef_left_1.stl" scale="0.001 0.001 0.001"/>
+      <mesh filename="file://$(find humanoid_final_copy_description)/meshes/eef_left_1.stl" scale="0.001 0.001 0.001"/>
     </geometry>
     <material name="silver"/>
@@ -280,5 +280,5 @@
     <origin xyz="-0.356985 0.180306 0.129143" rpy="0 0 0"/>
     <geometry>
-      <mesh filename="file:///home/ubuntu/ethr_rc_robot_assets/humanoid-description/humanoid_final_copy_description/meshes/eef_left_1.stl" scale="0.001 0.001 0.001"/>
+      <mesh filename="file://$(find humanoid_final_copy_description)/meshes/eef_left_1.stl" scale="0.001 0.001 0.001"/>
     </geometry>
   </collision>
@@ -293,5 +293,5 @@
     <origin xyz="0.191872 -0.059375 -0.229541" rpy="0 0 0"/>
     <geometry>
-      <mesh filename="file:///home/ubuntu/ethr_rc_robot_assets/humanoid-description/humanoid_final_copy_description/meshes/shoulder_upper_right_1.stl" scale="0.001 0.001 0.001"/>
+      <mesh filename="file://$(find humanoid_final_copy_description)/meshes/shoulder_upper_right_1.stl" scale="0.001 0.001 0.001"/>
     </geometry>
     <material name="silver"/>
@@ -300,5 +300,5 @@
     <origin xyz="0.191872 -0.059375 -0.229541" rpy="0 0 0"/>
     <geometry>
-      <mesh filename="file:///home/ubuntu/ethr_rc_robot_assets/humanoid-description/humanoid_final_copy_description/meshes/shoulder_upper_right_1.stl" scale="0.001 0.001 0.001"/>
+      <mesh filename="file://$(find humanoid_final_copy_description)/meshes/shoulder_upper_right_1.stl" scale="0.001 0.001 0.001"/>
     </geometry>
   </collision>
@@ -313,5 +313,5 @@
     <origin xyz="0.427833 0.119683 -0.130041" rpy="0 0 0"/>
     <geometry>
-      <mesh filename="file:///home/ubuntu/ethr_rc_robot_assets/humanoid-description/humanoid_final_copy_description/meshes/motor_2_right_1.stl" scale="0.001 0.001 0.001"/>
+      <mesh filename="file://$(find humanoid_final_copy_description)/meshes/motor_2_right_1.stl" scale="0.001 0.001 0.001"/>
     </geometry>
     <material name="silver"/>
@@ -320,5 +320,5 @@
     <origin xyz="0.427833 0.119683 -0.130041" rpy="0 0 0"/>
     <geometry>
-      <mesh filename="file:///home/ubuntu/ethr_rc_robot_assets/humanoid-description/humanoid_final_copy_description/meshes/motor_2_right_1.stl" scale="0.001 0.001 0.001"/>
+      <mesh filename="file://$(find humanoid_final_copy_description)/meshes/motor_2_right_1.stl" scale="0.001 0.001 0.001"/>
     </geometry>
   </collision>
@@ -333,5 +333,5 @@
     <origin xyz="0.236492 -0.021533 -0.261571" rpy="0 0 0"/>
     <geometry>
-      <mesh filename="file:///home/ubuntu/ethr_rc_robot_assets/humanoid-description/humanoid_final_copy_description/meshes/shoulder_lower_right_1.stl" scale="0.001 0.001 0.001"/>
+      <mesh filename="file://$(find humanoid_final_copy_description)/meshes/shoulder_lower_right_1.stl" scale="0.001 0.001 0.001"/>
     </geometry>
     <material name="silver"/>
@@ -340,5 +340,5 @@
     <origin xyz="0.236492 -0.021533 -0.261571" rpy="0 0 0"/>
     <geometry>
-      <mesh filename="file:///home/ubuntu/ethr_rc_robot_assets/humanoid-description/humanoid_final_copy_description/meshes/shoulder_lower_right_1.stl" scale="0.001 0.001 0.001"/>
+      <mesh filename="file://$(find humanoid_final_copy_description)/meshes/shoulder_lower_right_1.stl" scale="0.001 0.001 0.001"/>
     </geometry>
   </collision>
@@ -353,5 +353,5 @@
     <origin xyz="0.248948 -0.029004 -0.202053" rpy="0 0 0"/>
     <geometry>
-      <mesh filename="file:///home/ubuntu/ethr_rc_robot_assets/humanoid-description/humanoid_final_copy_description/meshes/motor_3_right_1.stl" scale="0.001 0.001 0.001"/>
+      <mesh filename="file://$(find humanoid_final_copy_description)/meshes/motor_3_right_1.stl" scale="0.001 0.001 0.001"/>
     </geometry>
     <material name="silver"/>
@@ -360,5 +360,5 @@
     <origin xyz="0.248948 -0.029004 -0.202053" rpy="0 0 0"/>
     <geometry>
-      <mesh filename="file:///home/ubuntu/ethr_rc_robot_assets/humanoid-description/humanoid_final_copy_description/meshes/motor_3_right_1.stl" scale="0.001 0.001 0.001"/>
+      <mesh filename="file://$(find humanoid_final_copy_description)/meshes/motor_3_right_1.stl" scale="0.001 0.001 0.001"/>
     </geometry>
   </collision>
@@ -373,5 +373,5 @@
     <origin xyz="0.272977 0.024558 -0.168884" rpy="0 0 0"/>
     <geometry>
-      <mesh filename="file:///home/ubuntu/ethr_rc_robot_assets/humanoid-description/humanoid_final_copy_description/meshes/elbow_upper_right_1.stl" scale="0.001 0.001 0.001"/>
+      <mesh filename="file://$(find humanoid_final_copy_description)/meshes/elbow_upper_right_1.stl" scale="0.001 0.001 0.001"/>
     </geometry>
     <material name="silver"/>
@@ -380,5 +380,5 @@
     <origin xyz="0.272977 0.024558 -0.168884" rpy="0 0 0"/>
     <geometry>
-      <mesh filename="file:///home/ubuntu/ethr_rc_robot_assets/humanoid-description/humanoid_final_copy_description/meshes/elbow_upper_right_1.stl" scale="0.001 0.001 0.001"/>
+      <mesh filename="file://$(find humanoid_final_copy_description)/meshes/elbow_upper_right_1.stl" scale="0.001 0.001 0.001"/>
     </geometry>
   </collision>
@@ -393,5 +393,5 @@
     <origin xyz="0.247858 0.043638 -0.074556" rpy="0 0 0"/>
     <geometry>
-      <mesh filename="file:///home/ubuntu/ethr_rc_robot_assets/humanoid-description/humanoid_final_copy_description/meshes/motor_4_right_1.stl" scale="0.001 0.001 0.001"/>
+      <mesh filename="file://$(find humanoid_final_copy_description)/meshes/motor_4_right_1.stl" scale="0.001 0.001 0.001"/>
     </geometry>
     <material name="silver"/>
@@ -400,5 +400,5 @@
     <origin xyz="0.247858 0.043638 -0.074556" rpy="0 0 0"/>
     <geometry>
-      <mesh filename="file:///home/ubuntu/ethr_rc_robot_assets/humanoid-description/humanoid_final_copy_description/meshes/motor_4_right_1.stl" scale="0.001 0.001 0.001"/>
+      <mesh filename="file://$(find humanoid_final_copy_description)/meshes/motor_4_right_1.stl" scale="0.001 0.001 0.001"/>
     </geometry>
   </collision>
@@ -413,5 +413,5 @@
     <origin xyz="0.311832 0.058966 -0.059764" rpy="0 0 0"/>
     <geometry>
-      <mesh filename="file:///home/ubuntu/ethr_rc_robot_assets/humanoid-description/humanoid_final_copy_description/meshes/elbow_lower_right_1.stl" scale="0.001 0.001 0.001"/>
+      <mesh filename="file://$(find humanoid_final_copy_description)/meshes/elbow_lower_right_1.stl" scale="0.001 0.001 0.001"/>
     </geometry>
     <material name="silver"/>
@@ -420,5 +420,5 @@
     <origin xyz="0.311832 0.058966 -0.059764" rpy="0 0 0"/>
     <geometry>
-      <mesh filename="file:///home/ubuntu/ethr_rc_robot_assets/humanoid-description/humanoid_final_copy_description/meshes/elbow_lower_right_1.stl" scale="0.001 0.001 0.001"/>
+      <mesh filename="file://$(find humanoid_final_copy_description)/meshes/elbow_lower_right_1.stl" scale="0.001 0.001 0.001"/>
     </geometry>
   </collision>
@@ -433,5 +433,5 @@
     <origin xyz="0.25945 0.098031 -0.014254" rpy="0 0 0"/>
     <geometry>
-      <mesh filename="file:///home/ubuntu/ethr_rc_robot_assets/humanoid-description/humanoid_final_copy_description/meshes/motor_5_right_1.stl" scale="0.001 0.001 0.001"/>
+      <mesh filename="file://$(find humanoid_final_copy_description)/meshes/motor_5_right_1.stl" scale="0.001 0.001 0.001"/>
     </geometry>
     <material name="silver"/>
@@ -440,5 +440,5 @@
     <origin xyz="0.25945 0.098031 -0.014254" rpy="0 0 0"/>
     <geometry>
-      <mesh filename="file:///home/ubuntu/ethr_rc_robot_assets/humanoid-description/humanoid_final_copy_description/meshes/motor_5_right_1.stl" scale="0.001 0.001 0.001"/>
+      <mesh filename="file://$(find humanoid_final_copy_description)/meshes/motor_5_right_1.stl" scale="0.001 0.001 0.001"/>
     </geometry>
   </collision>
@@ -453,5 +453,5 @@
     <origin xyz="0.299008 0.113647 0.03807" rpy="0 0 0"/>
     <geometry>
-      <mesh filename="file:///home/ubuntu/ethr_rc_robot_assets/humanoid-description/humanoid_final_copy_description/meshes/wrist_upper_right_1.stl" scale="0.001 0.001 0.001"/>
+      <mesh filename="file://$(find humanoid_final_copy_description)/meshes/wrist_upper_right_1.stl" scale="0.001 0.001 0.001"/>
     </geometry>
     <material name="silver"/>
@@ -460,5 +460,5 @@
     <origin xyz="0.299008 0.113647 0.03807" rpy="0 0 0"/>
     <geometry>
-      <mesh filename="file:///home/ubuntu/ethr_rc_robot_assets/humanoid-description/humanoid_final_copy_description/meshes/wrist_upper_right_1.stl" scale="0.001 0.001 0.001"/>
+      <mesh filename="file://$(find humanoid_final_copy_description)/meshes/wrist_upper_right_1.stl" scale="0.001 0.001 0.001"/>
     </geometry>
   </collision>
@@ -473,5 +473,5 @@
     <origin xyz="0.3034 0.098216 0.059827" rpy="0 0 0"/>
     <geometry>
-      <mesh filename="file:///home/ubuntu/ethr_rc_robot_assets/humanoid-description/humanoid_final_copy_description/meshes/motor_6_right_1.stl" scale="0.001 0.001 0.001"/>
+      <mesh filename="file://$(find humanoid_final_copy_description)/meshes/motor_6_right_1.stl" scale="0.001 0.001 0.001"/>
     </geometry>
     <material name="silver"/>
@@ -480,5 +480,5 @@
     <origin xyz="0.3034 0.098216 0.059827" rpy="0 0 0"/>
     <geometry>
-      <mesh filename="file:///home/ubuntu/ethr_rc_robot_assets/humanoid-description/humanoid_final_copy_description/meshes/motor_6_right_1.stl" scale="0.001 0.001 0.001"/>
+      <mesh filename="file://$(find humanoid_final_copy_description)/meshes/motor_6_right_1.stl" scale="0.001 0.001 0.001"/>
     </geometry>
   </collision>
@@ -493,5 +493,5 @@
     <origin xyz="0.303781 0.165604 0.057576" rpy="0 0 0"/>
     <geometry>
-      <mesh filename="file:///home/ubuntu/ethr_rc_robot_assets/humanoid-description/humanoid_final_copy_description/meshes/wrist_lower_right_1.stl" scale="0.001 0.001 0.001"/>
+      <mesh filename="file://$(find humanoid_final_copy_description)/meshes/wrist_lower_right_1.stl" scale="0.001 0.001 0.001"/>
     </geometry>
     <material name="silver"/>
@@ -500,5 +500,5 @@
     <origin xyz="0.303781 0.165604 0.057576" rpy="0 0 0"/>
     <geometry>
-      <mesh filename="file:///home/ubuntu/ethr_rc_robot_assets/humanoid-description/humanoid_final_copy_description/meshes/wrist_lower_right_1.stl" scale="0.001 0.001 0.001"/>
+      <mesh filename="file://$(find humanoid_final_copy_description)/meshes/wrist_lower_right_1.stl" scale="0.001 0.001 0.001"/>
     </geometry>
   </collision>
@@ -513,5 +513,5 @@
     <origin xyz="0.294907 0.140765 0.142689" rpy="0 0 0"/>
     <geometry>
-      <mesh filename="file:///home/ubuntu/ethr_rc_robot_assets/humanoid-description/humanoid_final_copy_description/meshes/motor_7_right_1.stl" scale="0.001 0.001 0.001"/>
+      <mesh filename="file://$(find humanoid_final_copy_description)/meshes/motor_7_right_1.stl" scale="0.001 0.001 0.001"/>
     </geometry>
     <material name="silver"/>
@@ -520,5 +520,5 @@
     <origin xyz="0.294907 0.140765 0.142689" rpy="0 0 0"/>
     <geometry>
-      <mesh filename="file:///home/ubuntu/ethr_rc_robot_assets/humanoid-description/humanoid_final_copy_description/meshes/motor_7_right_1.stl" scale="0.001 0.001 0.001"/>
+      <mesh filename="file://$(find humanoid_final_copy_description)/meshes/motor_7_right_1.stl" scale="0.001 0.001 0.001"/>
     </geometry>
   </collision>
@@ -533,5 +533,5 @@
     <origin xyz="0.353348 0.172025 0.130286" rpy="0 0 0"/>
     <geometry>
-      <mesh filename="file:///home/ubuntu/ethr_rc_robot_assets/humanoid-description/humanoid_final_copy_description/meshes/eef_right_1.stl" scale="0.001 0.001 0.001"/>
+      <mesh filename="file://$(find humanoid_final_copy_description)/meshes/eef_right_1.stl" scale="0.001 0.001 0.001"/>
     </geometry>
     <material name="silver"/>
@@ -540,5 +540,5 @@
     <origin xyz="0.353348 0.172025 0.130286" rpy="0 0 0"/>
     <geometry>
-      <mesh filename="file:///home/ubuntu/ethr_rc_robot_assets/humanoid-description/humanoid_final_copy_description/meshes/eef_right_1.stl" scale="0.001 0.001 0.001"/>
+      <mesh filename="file://$(find humanoid_final_copy_description)/meshes/eef_right_1.stl" scale="0.001 0.001 0.001"/>
     </geometry>
   </collision>
@@ -553,5 +553,5 @@
     <origin xyz="0.173947 -0.09865 -0.225664" rpy="0 0 0"/>
     <geometry>
-      <mesh filename="file:///home/ubuntu/ethr_rc_robot_assets/humanoid-description/humanoid_final_copy_description/meshes/motor_1_right_1.stl" scale="0.001 0.001 0.001"/>
+      <mesh filename="file://$(find humanoid_final_copy_description)/meshes/motor_1_right_1.stl" scale="0.001 0.001 0.001"/>
     </geometry>
     <material name="silver"/>
@@ -560,5 +560,5 @@
     <origin xyz="0.173947 -0.09865 -0.225664" rpy="0 0 0"/>
     <geometry>
-      <mesh filename="file:///home/ubuntu/ethr_rc_robot_assets/humanoid-description/humanoid_final_copy_description/meshes/motor_1_right_1.stl" scale="0.001 0.001 0.001"/>
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